File: crc/2026-Node/2026-Node.kicad_pcb (KiCad board)
At the start: 2 copper layers, 32.6 x 83.4 mm, 24 parts, among them J1 Conn_01x02, J2 Conn_01x02, J3 Conn_01x04, J4 Conn_01x04, J5 Conn_01x04, J6 Conn_01x04, J7 Conn_01x04, J8 Conn_01x06, SW1 SW_MEC_5E, U1 STM32F446RETx, U2 NJM2845DL1-33-TE1, U3 MCP2561-E-SN, U4 MCP2561-E-SN, Y1 Crystal_GND24_Small

Commit message: MDSUBのガーバー再生成
Parts:
- added C1: 0.1uF, Capacitor_SMD:C_0603_1608Metric_Pad1.08x0.95mm_HandSolder, F.Cu at (117.5, 78.5)
- added C2: 20pf, Capacitor_SMD:C_0603_1608Metric_Pad1.08x0.95mm_HandSolder, F.Cu at (112.6, 90.5)
- added C3: 20pf, Capacitor_SMD:C_0603_1608Metric_Pad1.08x0.95mm_HandSolder, F.Cu at (114.4, 90.5)
- added C4: 0.1uF, Capacitor_SMD:C_0603_1608Metric_Pad1.08x0.95mm_HandSolder, F.Cu at (127.0, 112.7)
- added C5: 0.1uF, Capacitor_SMD:C_0603_1608Metric_Pad1.08x0.95mm_HandSolder, F.Cu at (131.5, 112.6)
- added C6: 1uF, Capacitor_SMD:C_0603_1608Metric_Pad1.08x0.95mm_HandSolder, F.Cu at (126.1, 96.1)
- added J1: Conn_01x02, Connector_PinHeader_2.54mm:PinHeader_1x02_P2.54mm_Vertical, F.Cu at (115.2, 64.4)
- added J2: Conn_01x02, Connector_PinHeader_2.54mm:PinHeader_1x02_P2.54mm_Vertical, F.Cu at (113.7, 99.8)
- added J3: Conn_01x04, Connector_JST:JST_XH_B4B-XH-A_1x04_P2.50mm_Vertical, F.Cu at (136.1, 43.5)
- added J4: Conn_01x04, Connector_JST:JST_XH_S4B-XH-A_1x04_P2.50mm_Horizontal, F.Cu at (121.3, 36.3)
- added J5: Conn_01x04, Connector_JST:JST_XH_B4B-XH-A_1x04_P2.50mm_Vertical, F.Cu at (121.3, 43.6)
- added J6: Conn_01x04, Connector_JST:JST_XH_S4B-XH-A_1x04_P2.50mm_Horizontal, F.Cu at (136.1, 36.2)
- added J7: Conn_01x04, Connector_JST:JST_XH_S4B-XH-A_1x04_P2.50mm_Horizontal, F.Cu at (112.7, 107.9)
- added J8: Conn_01x06, Connector_PinHeader_2.54mm:PinHeader_1x06_P2.54mm_Vertical, F.Cu at (138.8, 68.7)
- added R1: 470, Resistor_SMD:R_0603_1608Metric_Pad0.98x0.95mm_HandSolder, F.Cu at (117.5, 74.3)
- added R2: 10k, Resistor_SMD:R_0603_1608Metric_Pad0.98x0.95mm_HandSolder, F.Cu at (121.7, 78.5)
- added R3: 120, Resistor_SMD:R_0603_1608Metric_Pad0.98x0.95mm_HandSolder, F.Cu at (129.4, 64.3)
- added R4: R, Resistor_SMD:R_0603_1608Metric_Pad0.98x0.95mm_HandSolder, F.Cu at (113.7, 96.5)
- added SW1: SW_MEC_5E, SKRPABE010:SW4_SKRPABE010_ALPS, F.Cu at (113.5, 76.4)
- added U1: STM32F446RETx, Package_QFP:LQFP-64_10x10mm_P0.5mm, F.Cu at (122.5, 86.7)
- added U2: NJM2845DL1-33-TE1, NJM2845DL1-33-TE1:DPAK228P968X238-4N, F.Cu at (130.1, 105.7)
- added U3: MCP2561-E-SN, Package_SO:SOIC-8_3.9x4.9mm_P1.27mm, F.Cu at (124.3, 68.7)
- added U4: MCP2561-E-SN, Package_SO:SOIC-8_3.9x4.9mm_P1.27mm, F.Cu at (121.3, 101.4)
- added Y1: Crystal_GND24_Small, TSX_3225_25_0000MF10P_C0:XTAL_TSX-3225_25.0000MF10P-C0, F.Cu at (113.0, 85.2)
- moved C10 16.3 mm to (159.6, 112.7)
- moved C11 16.3 mm to (164.2, 112.6)
- moved C12 16.3 mm to (158.7, 96.1)
- moved C7 16.3 mm to (150.1, 78.5)
- moved C8 16.3 mm to (145.3, 90.5)
- moved C9 16.3 mm to (147.0, 90.5)
- moved J10 16.3 mm to (146.4, 99.8)
- moved J11 16.3 mm to (168.7, 43.5)
- moved J12 16.3 mm to (153.9, 36.3)
- moved J13 16.3 mm to (153.9, 43.6)
- moved J14 16.3 mm to (168.7, 36.2)
- moved J15 16.3 mm to (145.4, 107.9)
- moved J16 16.3 mm to (171.4, 68.7)
- moved J9 16.3 mm to (147.9, 64.4)
- moved R5 16.3 mm to (150.1, 74.3)
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- renumbered C4 to C10, C5 to C11, C6 to C12, C1 to C7, C2 to C8, C3 to C9, J2 to J10, J3 to J11, J4 to J12, J5 to J13, J6 to J14, J7 to J15, J8 to J16, J1 to J9, R1 to R5, R2 to R6, R3 to R7, R4 to R8, SW1 to SW2, U1 to U5, U2 to U6, U3 to U7, U4 to U8, Y1 to Y2
Routing:
- net +5V: track 175.3 -> 350.5 mm
- net CAN1_L: track 101.4 -> 202.7 mm
- net +3.3V: track 93.8 -> 187.6 mm, vias 2 -> 4
- net CAN1_H: track 90.9 -> 181.8 mm, vias 3 -> 6
- net NRST: track 36.8 -> 73.5 mm
- net CAN1_TX: track 30.0 -> 60.1 mm, vias 2 -> 4
- net SWO: track 23.2 -> 46.5 mm, vias 2 -> 4
- net CAN2_TX: track 18.0 -> 36.1 mm
- net SWDIO: track 17.7 -> 35.4 mm, vias 2 -> 4
- net CAN1_RX: track 17.4 -> 34.9 mm, vias 2 -> 4
- net CAN2_L: track 16.7 -> 33.5 mm
- net CAN2_H: track 15.8 -> 31.5 mm
- net Net-(J1-Pin_2): track 14.8 -> 29.6 mm
- net GND: track 14.7 -> 29.3 mm, vias 497 -> 994
- net CAN2_RX: track 13.8 -> 27.7 mm
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Other:
- board size 32.6 x 83.4 mm -> 65.2 x 83.4 mm
