File: crc/ISS_MD_SUB/ISS_MD_SUB.kicad_pcb (KiCad board)
At the start: 2 copper layers, 67.5 x 75 mm, 60 parts, among them J1 Conn_01x06, J10 Enc, J11 Conn_01x02, J12 Conn_01x02, J13 Conn_01x10, J14 Conn_01x02, J2 Conn_01x04, J3 Enc, J4 Conn_01x02, J5 Conn_01x02, J6 Conn_01x10, J7 Conn_01x02, J8 Conn_01x06, J9 Conn_01x04, SW1 SW_MEC_5E, SW2 SW_DIP_x03, SW3 SW_MEC_5E, SW4 SW_DIP_x03, U1 STM32F303K8Tx, U2 NJM2845DL1-33-TE1, U3 MCP2561-E-SN, U4 STM32F303K8Tx, U5 NJM2845DL1-33-TE1, U6 MCP2561-E-SN, Y1 Crystal_GND24_Small, Y2 Crystal_GND24_Small

Commit message: ノード完成
Parts:
- removed the C3 at (101.7, 112.7)
- removed the C4 at (97.5, 120.8)
- removed D1: LED, LED_SMD:LED_0603_1608Metric_Pad1.05x0.95mm_HandSolder
- removed J1: Conn_01x06, Connector_PinHeader_2.54mm:PinHeader_1x06_P2.54mm_Vertical
- removed the J3 at (99.0, 75.5)
- removed the J5 at (109.0, 75.9)
- removed R1, R2: 10k, Resistor_SMD:R_0603_1608Metric_Pad0.98x0.95mm_HandSolder
- removed the R10 at (107.8, 138.6)
- removed the R5 at (119.1, 125.2)
- removed the R6 at (118.3, 82.4)
- removed R7, R8: 1k, Resistor_SMD:R_0603_1608Metric_Pad0.98x0.95mm_HandSolder
- removed SW1: SW_MEC_5E, SKRPABE010:SW4_SKRPABE010_ALPS
- removed the U2 at (101.1, 125.9)
- added C8: 20pF, Capacitor_SMD:C_0603_1608Metric_Pad1.08x0.95mm_HandSolder, F.Cu at (118.5, 112.7)
- added C9: 0.1uF, Capacitor_SMD:C_0603_1608Metric_Pad1.08x0.95mm_HandSolder, F.Cu at (114.4, 120.8)
- added D3: LED, LED_SMD:LED_0603_1608Metric_Pad1.05x0.95mm_HandSolder, F.Cu at (140.8, 137.4)
- added J10: Enc, Connector_JST:JST_XH_S4B-XH-A_1x04_P2.50mm_Horizontal, F.Cu at (116.0, 75.5)
- added J12: Conn_01x02, Connector_JST:JST_XH_B2B-XH-A_1x02_P2.50mm_Vertical, F.Cu at (125.9, 75.9)
- added J8: Conn_01x06, Connector_PinHeader_2.54mm:PinHeader_1x06_P2.54mm_Vertical, F.Cu at (141.3, 100.0)
- added R11: 10k, Resistor_SMD:R_0603_1608Metric_Pad0.98x0.95mm_HandSolder, F.Cu at (118.8, 102.6)
- added R12: 10k, Resistor_SMD:R_0603_1608Metric_Pad0.98x0.95mm_HandSolder, F.Cu at (119.9, 99.3)
- added R15: 120, Resistor_SMD:R_0603_1608Metric_Pad0.98x0.95mm_HandSolder, F.Cu at (136.0, 125.2)
- added R16: 1k, Resistor_SMD:R_0603_1608Metric_Pad0.98x0.95mm_HandSolder, F.Cu at (135.2, 82.4)
- added R17: 1k, Resistor_SMD:R_0603_1608Metric_Pad0.98x0.95mm_HandSolder, F.Cu at (125.9, 81.8)
- added R18: 1k, Resistor_SMD:R_0603_1608Metric_Pad0.98x0.95mm_HandSolder, B.Cu at (121.3, 138.6)
- added R20: 1k, Resistor_SMD:R_0603_1608Metric_Pad0.98x0.95mm_HandSolder, B.Cu at (124.8, 138.6)
- added SW3: SW_MEC_5E, SKRPABE010:SW4_SKRPABE010_ALPS, F.Cu at (114.7, 100.5)
- added U5: NJM2845DL1-33-TE1, NJM2845DL1-33-TE1:DPAK228P968X238-4N, F.Cu at (118.0, 125.9)
- D2, D4: value CAN_LED -> LED
- SW2, SW4: footprint Button_Switch_SMD:SW_DIP_SPSTx03_Slide_6.7x9.18mm_W6.73mm_P2.54mm_LowProfile_JPin -> Button_Switch_THT:SW_DIP_SPSTx03_Slide_9.78x9.8mm_W7.62mm_P2.54mm
- moved C1 16.9 mm to (117.9, 99.3)
- moved C10 16.9 mm to (152.3, 112.7)
- moved C11 16.9 mm to (148.2, 120.8)
- moved C3 16.9 mm to (151.7, 99.3)
- moved C4 16.9 mm to (154.3, 112.7)
- moved C5 16.9 mm to (112.7, 120.8)
- moved C6 16.9 mm to (146.5, 120.8)
- moved D2 16.9 mm to (140.9, 130.2)
- moved D5 16.9 mm to (174.7, 137.4)
- moved J11 16.9 mm to (164.1, 121.7)
- moved J13 16.9 mm to (175.1, 100.0)
- moved J14 16.9 mm to (149.8, 75.5)
- moved J15 16.9 mm to (159.7, 75.9)
- moved J2 16.9 mm to (113.3, 134.4)
- moved J5 16.9 mm to (170.5, 75.6)
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- renumbered C8 to C10, C9 to C11, C6 to C3, C7 to C4, C10 to C6, D3 to D5, J14 to J11, J8 to J13, J10 to J14, J12 to J15, J9 to J3, J11 to J5, J13 to J9, R19 to R10, R11 to R13, R12 to R14, R15 to R19, R16 to R21, R17 to R22, R18 to R23, R20 to R24, R13 to R5, R14 to R6, SW3 to SW5, U4 to U2, U6 to U4, U5 to U6
Routing:
- net ID1: track 66.7 -> 70.5 mm
- net ID2: track 73.4 -> 75.0 mm, vias 8 -> 6
- net ID3: track 71.9 -> 73.3 mm, vias 2 -> 0
- net GND: vias 1260 -> 1250
Other:
- outline, holes or cut-outs redrawn
